File: 1. LED Chaser Circuit/1. LED Chaser Circuit.kicad_sch (KiCad schematic)
At the start: 19 parts, among them U1 NE555D, U2 4017

Commit message: Add files via upload
Parts:
- U2: footprint (none) -> Package_DIP:DIP-16_W10.16mm
Changed lines of the file:
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@@
 			)
 		)
-		(property "Footprint" ""
+		(property "Footprint" "Package_DIP:DIP-16_W10.16mm"
 			(at 171.45 87.63 0)
 			(hide yes)
